File: hardware/bus_power_switch/bus_power.brd (EAGLE design)
At the start: 25.4 x 33 mm, 12 parts, among them Q1 IRF4905, Q2 IRF4905, Q3 BSS138, Q4 BSS138, X1 MKDSN1,5/2-5,08, X2 MKDSN1,5/2-5,08, X3 MKDSN1,5/2-5,08

Commit message: changed some resistor values
Parts:
- R1: value 1k5 -> 1k
Changed lines of the file:
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@@
 <element name="Q1" library="transistor-power" package="TO220BV" value="IRF4905" x="13.97" y="6.35" smashed="yes" rot="R270"/>
 <element name="Q2" library="transistor-power" package="TO220BV" value="IRF4905" x="13.97" y="26.67" smashed="yes" rot="R270"/>
-<element name="R1" library="rcl" package="R0805" value="1k5" x="15.24" y="6.35" smashed="yes" rot="MR270"/>
+<element name="R1" library="rcl" package="R0805" value="1k" x="15.24" y="6.35" smashed="yes" rot="MR270"/>
 <element name="R2" library="rcl" package="R0805" value="1k5" x="15.24" y="26.67" smashed="yes" rot="MR270"/>
 <element name="Q3" library="transistor-small-signal" package="SOT23" value="BSS138" x="17.78" y="10.16" smashed="yes" rot="MR270"/>
