File: hardware/bus_power_switch/bus_power.sch (EAGLE design)
At the start: 12 parts, among them Q1 IRF4905, Q2 IRF4905, Q3 BSS138, Q4 BSS138, X1 MKDSN1,5/2-5,08, X2 MKDSN1,5/2-5,08, X3 MKDSN1,5/2-5,08

Commit message: changed some resistor values
Parts:
- R1: value 1k5 -> 1k
Changed lines of the file:
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@@
 <part name="P+1" library="supply1" deviceset="+12V" device=""/>
 <part name="P+2" library="supply1" deviceset="+5V" device=""/>
-<part name="R1" library="rcl" deviceset="R-EU_" device="R0805" value="1k5"/>
+<part name="R1" library="rcl" deviceset="R-EU_" device="R0805" value="1k"/>
 <part name="R2" library="rcl" deviceset="R-EU_" device="R0805" value="1k5"/>
 <part name="P+3" library="supply1" deviceset="+5V" device=""/>
