File: hardware/DALI_interface/DALI_Master.sch (EAGLE design)
At the start: 25 parts, among them IC1 LM393D, Q1 BD135, Q2 BC817-25, Q3 BC817-25, X1 MKDSN1,5/2-5,08, X2 MKDSN1,5/2-5,08

Commit message: added the missing resistor values and a reference to the site with the original idea
Parts:
- R10, R11: value (none) -> 1k
- R7: value (none) -> 470R
Other:
- note added: "idea taken from: http://zerties.org/index.php/DALI"
Changed lines of the file:
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@@
 <part name="GND3" library="supply1" deviceset="GND" device=""/>
 <part name="GND4" library="supply1" deviceset="GND" device=""/>
-<part name="R7" library="rcl" deviceset="R-EU_" device="R0805"/>
+<part name="R7" library="rcl" deviceset="R-EU_" device="R0805" value="470R"/>
 <part name="R8" library="rcl" deviceset="R-EU_" device="R1206" value="5R6"/>
 <part name="R9" library="rcl" deviceset="R-EU_" device="R1206" value="5R6"/>
@@
 <part name="D1" library="diode" deviceset="BAT54S" device=""/>
 <part name="P+10" library="supply1" deviceset="+12V" device=""/>
-<part name="R10" library="rcl" deviceset="R-EU_" device="R0805"/>
+<part name="R10" library="rcl" deviceset="R-EU_" device="R0805" value="1k"/>
 <part name="C4" library="rcl" deviceset="CPOL-EU" device="E2.5-6" value="100u"/>
 <part name="P+11" library="supply1" deviceset="+5V" device=""/>
-<part name="R11" library="rcl" deviceset="R-EU_" device="R0805"/>
+<part name="R11" library="rcl" deviceset="R-EU_" device="R0805" value="1k"/>
 <part name="GND5" library="supply1" deviceset="GND" device=""/>
 <part name="P+12" library="supply1" deviceset="+12V" device=""/>
@@
 <sheet>
 <plain>
-<text x="76.2" y="30.48" size="1.778" layer="97">led off -&gt; bus not active</text>
+<text x="63.5" y="30.48" size="1.778" layer="97">led off -&gt; bus not active</text>
+<text x="66.04" y="2.54" size="1.778" layer="97">idea taken from: http://zerties.org/index.php/DALI</text>
 </plain>
 <instances>
@@
 <instance part="R5" gate="G$1" x="48.26" y="30.48" rot="R90"/>
 <instance part="GND4" gate="1" x="91.44" y="10.16"/>
-<instance part="R7" gate="G$1" x="96.52" y="20.32"/>
+<instance part="R7" gate="G$1" x="91.44" y="27.94" rot="R90"/>
 <instance part="R8" gate="G$1" x="30.48" y="7.62" rot="R90"/>
 <instance part="R9" gate="G$1" x="22.86" y="7.62" rot="R90"/>
@@
 <instance part="OK3" gate="G$1" x="68.58" y="55.88"/>
 <instance part="OK4" gate="G$1" x="78.74" y="17.78" rot="MR0"/>
+<instance part="SV1" gate="G$1" x="111.76" y="53.34" rot="MR180"/>
+<instance part="C1" gate="G$1" x="93.98" y="71.12"/>
+<instance part="P+1" gate="1" x="96.52" y="43.18" rot="R90"/>
+<instance part="P+2" gate="1" x="127" y="43.18" rot="MR90"/>
+<instance part="P+3" gate="1" x="93.98" y="76.2"/>
+<instance part="GND1" gate="1" x="121.92" y="35.56"/>
+<instance part="GND2" gate="1" x="101.6" y="35.56"/>
+<instance part="GND3" gate="1" x="93.98" y="63.5"/>
 </instances>
 <busses>
@@
 <pinref part="GND5" gate="1" pin="GND"/>
 </segment>
+<segment>
+<pinref part="SV1" gate="G$1" pin="20"/>
+<wire x1="119.38" y1="40.64" x2="121.92" y2="40.64" width="0.1524" layer="91"/>
+<wire x1="121.92" y1="40.64" x2="121.92" y2="38.1" width="0.1524" layer="91"/>
+<pinref part="GND1" gate="1" pin="GND"/>
+</segment>
+<segment>
+<wire x1="104.14" y1="40.64" x2="101.6" y2="40.64" width="0.1524" layer="91"/>
+<wire x1="101.6" y1="40.64" x2="101.6" y2="38.1" width="0.1524" layer="91"/>
+<pinref part="SV1" gate="G$1" pin="19"/>
+<pinref part="GND2" gate="1" pin="GND"/>
+</segment>
+<segment>
+<pinref part="C1" gate="G$1" pin="2"/>
+<pinref part="GND3" gate="1" pin="GND"/>
+</segment>
 </net>
 <net name="N$10" class="0">
 <segment>
 <pinref part="R7" gate="G$1" pin="1"/>
+<wire x1="91.44" y1="22.86" x2="91.44" y2="20.32" width="0.1524" layer="91"/>
 <wire x1="91.44" y1="20.32" x2="88.9" y2="20.32" width="0.1524" layer="91"/>
 <pinref part="OK4" gate="G$1" pin="A"/>
@@
 <net name="DALI_TX" class="0">
 <segment>
+<pinref part="SV1" gate="G$1" pin="11"/>
+<wire x1="104.14" y1="50.8" x2="91.44" y2="50.8" width="0.1524" layer="91"/>
+<label x="91.44" y="50.8" size="1.778" layer="95"/>
 <pinref part="R7" gate="G$1" pin="2"/>
-<wire x1="101.6" y1="20.32" x2="111.76" y2="20.32" width="0.1524" layer="91"/>
-<label x="101.6" y="20.32" size="1.778" layer="95"/>
+<wire x1="91.44" y1="33.02" x2="91.44" y2="50.8" width="0.1524" layer="91"/>
 </segment>
 </net>
@@
 <pinref part="OK3" gate="G$1" pin="COL"/>
 </segment>
+<segment>
+<wire x1="99.06" y1="43.18" x2="104.14" y2="43.18" width="0.1524" layer="91"/>
+<pinref part="SV1" gate="G$1" pin="17"/>
+<pinref part="P+1" gate="1" pin="+5V"/>
+</segment>
+<segment>
+<pinref part="SV1" gate="G$1" pin="18"/>
+<wire x1="119.38" y1="43.18" x2="124.46" y2="43.18" width="0.1524" layer="91"/>
+<pinref part="P+2" gate="1" pin="+5V"/>
+</segment>
+<segment>
+<pinref part="C1" gate="G$1" pin="1"/>
+<pinref part="P+3" gate="1" pin="+5V"/>
+</segment>
 </net>
 <net name="DALI_RX" class="0">
@@
 <wire x1="76.2" y1="53.34" x2="78.74" y2="53.34" width="0.1524" layer="91"/>
 <wire x1="78.74" y1="53.34" x2="78.74" y2="50.8" width="0.1524" layer="91"/>
-<wire x1="78.74" y1="53.34" x2="91.44" y2="53.34" width="0.1524" layer="91"/>
+<wire x1="78.74" y1="53.34" x2="104.14" y2="53.34" width="0.1524" layer="91"/>
 <junction x="78.74" y="53.34"/>
-<label x="81.28" y="53.34" size="1.778" layer="95"/>
 <pinref part="OK3" gate="G$1" pin="EMIT"/>
+<pinref part="SV1" gate="G$1" pin="9"/>
+<label x="91.44" y="53.34" size="1.778" layer="95"/>
 </segment>
 </net>
@@
 </segment>
 </net>
-</nets>
-</sheet>
-<sheet>
-<plain>
-</plain>
-<instances>
-<instance part="SV1" gate="G$1" x="27.94" y="20.32" rot="MR180"/>
-<instance part="C1" gate="G$1" x="17.78" y="53.34"/>
-<instance part="P+1" gate="1" x="12.7" y="10.16" rot="R90"/>
-<instance part="P+2" gate="1" x="43.18" y="10.16" rot="MR90"/>
-<instance part="P+3" gate="1" x="17.78" y="58.42"/>
-<instance part="GND1" gate="1" x="38.1" y="2.54"/>
-<instance part="GND2" gate="1" x="17.78" y="2.54"/>
-<instance part="GND3" gate="1" x="17.78" y="45.72"/>
-</instances>
-<busses>
-</busses>
-<nets>
-<net name="+5V" class="0">
-<segment>
-<wire x1="15.24" y1="10.16" x2="20.32" y2="10.16" width="0.1524" layer="91"/>
-<pinref part="SV1" gate="G$1" pin="17"/>
-<pinref part="P+1" gate="1" pin="+5V"/>
-</segment>
-<segment>
-<pinref part="SV1" gate="G$1" pin="18"/>
-<wire x1="35.56" y1="10.16" x2="40.64" y2="10.16" width="0.1524" layer="91"/>
-<pinref part="P+2" gate="1" pin="+5V"/>
-</segment>
-<segment>
-<pinref part="C1" gate="G$1" pin="1"/>
-<pinref part="P+3" gate="1" pin="+5V"/>
-</segment>
-</net>
-<net name="DALI_TX" class="0">
-<segment>
-<pinref part="SV1" gate="G$1" pin="11"/>
-<wire x1="20.32" y1="17.78" x2="7.62" y2="17.78" width="0.1524" layer="91"/>
-<label x="7.62" y="17.78" size="1.778" layer="95"/>
-</segment>
-</net>
-<net name="DALI_RX" class="0">
-<segment>
-<pinref part="SV1" gate="G$1" pin="9"/>
-<wire x1="20.32" y1="20.32" x2="7.62" y2="20.32" width="0.1524" layer="91"/>
-<label x="7.62" y="20.32" size="1.778" layer="95"/>
-</segment>
-</net>
-<net name="GND" class="0">
-<segment>
-<pinref part="SV1" gate="G$1" pin="20"/>
-<wire x1="35.56" y1="7.62" x2="38.1" y2="7.62" width="0.1524" layer="91"/>
-<wire x1="38.1" y1="7.62" x2="38.1" y2="5.08" width="0.1524" layer="91"/>
-<pinref part="GND1" gate="1" pin="GND"/>
-</segment>
-<segment>
-<wire x1="20.32" y1="7.62" x2="17.78" y2="7.62" width="0.1524" layer="91"/>
-<wire x1="17.78" y1="7.62" x2="17.78" y2="5.08" width="0.1524" layer="91"/>
-<pinref part="SV1" gate="G$1" pin="19"/>
-<pinref part="GND2" gate="1" pin="GND"/>
-</segment>
-<segment>
-<pinref part="C1" gate="G$1" pin="2"/>
-<pinref part="GND3" gate="1" pin="GND"/>
-</segment>
-</net>

Commit message: changed some resistor values
Parts:
- R10: value 1k -> 1k5
Changed lines of the file:
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@@
 <part name="D1" library="diode" deviceset="BAT54S" device=""/>
 <part name="P+10" library="supply1" deviceset="+12V" device=""/>
-<part name="R10" library="rcl" deviceset="R-EU_" device="R0805" value="1k"/>
+<part name="R10" library="rcl" deviceset="R-EU_" device="R0805" value="1k5"/>
 <part name="C4" library="rcl" deviceset="CPOL-EU" device="E2.5-6" value="100u"/>
 <part name="P+11" library="supply1" deviceset="+5V" device=""/>

Commit message: change the value of the capacitor on the bus to be in spec
Parts:
- C3: value 220n -> 100n
Changed lines of the file:
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@@
 <part name="AGND8" library="supply1" deviceset="AGND" device=""/>
 <part name="AGND9" library="supply1" deviceset="AGND" device=""/>
-<part name="C3" library="rcl" deviceset="C-EU" device="C0805" value="220n"/>
+<part name="C3" library="rcl" deviceset="C-EU" device="C0805" value="100n"/>
 <part name="D1" library="diode" deviceset="BAT54S" device=""/>
 <part name="P+10" library="supply1" deviceset="+12V" device=""/>
