File: hardware/busfahrer_pi/direct/busfahrer_pi.sch (EAGLE design)
At the start: 21 parts, among them Q1 20 MHz, X1 MKDSN1,5/2-5,08

Commit message: some fixes
Parts:
- C3, C4: value 15p -> 22p
- R4: device rcl:R-EU_R0805 -> rcl_patch:R-EU_R0805
- R6, R7: value 220 -> 330
Connections:
- net N$5 renamed TXCAN
- removed net N$6: MCP2515D.RXCAN, R4.2, R5.1
- removed net N$7: MCP2551G$1.RXD, R4.1
- new net RXCAN: MCP2515D.RXCAN, R4.1, R5.1
- new net RXCAN_5V: MCP2551G$1.RXD, R4.2
- net +3V3: now also MCP2515D.RESET; no longer R1.2
- net GND: now also R1.1; no longer MCP2551G$1.RS
- net N$1: now also MCP2551G$1.RS, R1.2; no longer MCP2515D.RESET, R1.1
Other:
- moved on the sheet: R1, R2, R3, R4
Changed lines of the file:
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@@
 <?xml version="1.0" encoding="utf-8"?>
 <!DOCTYPE eagle SYSTEM "eagle.dtd">
-<eagle version="6.1">
+<eagle version="6.4">
 <drawing>
 <settings>
@@
 <part name="GND10" library="supply1" deviceset="GND" device=""/>
 <part name="+3V4" library="supply1" deviceset="+3V3" device=""/>
-<part name="R1" library="rcl" deviceset="R-EU_" device="R0805" value="10k"/>
 <part name="R2" library="rcl" deviceset="R-EU_" device="R0805" value="10k"/>
 <part name="R3" library="rcl" deviceset="R-EU_" device="R0805" value="10k"/>
 <part name="C1" library="rcl" deviceset="C-EU" device="C0805" value="100n"/>
 <part name="C2" library="rcl" deviceset="C-EU" device="C0805" value="100n"/>
-<part name="C3" library="rcl" deviceset="C-EU" device="C0805" value="15p"/>
-<part name="C4" library="rcl" deviceset="C-EU" device="C0805" value="15p"/>
+<part name="C3" library="rcl" deviceset="C-EU" device="C0805" value="22p"/>
+<part name="C4" library="rcl" deviceset="C-EU" device="C0805" value="22p"/>
 <part name="GND12" library="supply1" deviceset="GND" device=""/>
 <part name="Q1" library="crystal" deviceset="CRYSTAL" device="HC49S" value="20 MHz"/>
 <part name="GND13" library="supply1" deviceset="GND" device=""/>
-<part name="R4" library="rcl" deviceset="R-EU_" device="R0805" value="10k"/>
 <part name="R5" library="rcl" deviceset="R-EU_" device="R0805" value="18k"/>
 <part name="GND14" library="supply1" deviceset="GND" device=""/>
-<part name="R6" library="rcl" deviceset="R-EU_" device="R0805" value="220"/>
-<part name="R7" library="rcl" deviceset="R-EU_" device="R0805" value="220"/>
+<part name="R6" library="rcl" deviceset="R-EU_" device="R0805" value="330"/>
+<part name="R7" library="rcl" deviceset="R-EU_" device="R0805" value="330"/>
 <part name="LED1" library="led" deviceset="LED" device="CHIP-LED0805"/>
 <part name="LED2" library="led" deviceset="LED" device="CHIP-LED0805"/>
 <part name="GND11" library="supply1" deviceset="GND" device=""/>
 <part name="C5" library="rcl" deviceset="CPOL-EU" device="E2.5-6" value="100u"/>
+<part name="R4" library="rcl_patch" deviceset="R-EU_" device="R0805" value="10k"/>
+<part name="+3V5" library="supply1" deviceset="+3V3" device=""/>
+<part name="R1" library="rcl" deviceset="R-EU_" device="R0805" value="10k"/>
 </parts>
 <sheets>
@@
 <instance part="SV3" gate="G$1" x="170.18" y="96.52" rot="R180"/>
 <instance part="GND10" gate="1" x="160.02" y="96.52" rot="R270"/>
-<instance part="+3V4" gate="G$1" x="45.72" y="81.28"/>
-<instance part="R1" gate="G$1" x="45.72" y="71.12" rot="R90"/>
-<instance part="R2" gate="G$1" x="38.1" y="71.12" rot="R90"/>
-<instance part="R3" gate="G$1" x="30.48" y="71.12" rot="R90"/>
+<instance part="+3V4" gate="G$1" x="38.1" y="78.74"/>
+<instance part="R2" gate="G$1" x="38.1" y="66.04" rot="R90"/>
+<instance part="R3" gate="G$1" x="30.48" y="66.04" rot="R90"/>
 <instance part="C1" gate="G$1" x="60.96" y="96.52"/>
 <instance part="C2" gate="G$1" x="78.74" y="96.52"/>
@@
 <instance part="GND12" gate="1" x="40.64" y="17.78"/>
 <instance part="Q1" gate="G$1" x="40.64" y="33.02" rot="R180"/>
-<instance part="GND13" gate="1" x="114.3" y="43.18"/>
-<instance part="R4" gate="G$1" x="109.22" y="55.88" rot="R180"/>
+<instance part="GND13" gate="1" x="114.3" y="33.02"/>
 <instance part="R5" gate="G$1" x="101.6" y="48.26" rot="R270"/>
 <instance part="GND14" gate="1" x="101.6" y="38.1"/>
@@
 <instance part="GND11" gate="1" x="91.44" y="7.62"/>
 <instance part="C5" gate="G$1" x="88.9" y="96.52"/>
+<instance part="R4" gate="G$1" x="109.22" y="55.88"/>
+<instance part="+3V5" gate="G$1" x="45.72" y="68.58"/>
+<instance part="R1" gate="G$1" x="114.3" y="43.18" rot="R90"/>
 </instances>
 <busses>
@@
 </segment>
 <segment>
-<pinref part="MCP2551" gate="G$1" pin="RS"/>
-<pinref part="GND13" gate="1" pin="GND"/>
-<wire x1="116.84" y1="48.26" x2="114.3" y2="48.26" width="0.1524" layer="91"/>
-<wire x1="114.3" y1="48.26" x2="114.3" y2="45.72" width="0.1524" layer="91"/>
-</segment>
-<segment>
 <pinref part="LED1" gate="G$1" pin="C"/>
 <wire x1="86.36" y1="15.24" x2="86.36" y2="12.7" width="0.1524" layer="91"/>
@@
 <junction x="91.44" y="12.7"/>
 </segment>
+<segment>
+<pinref part="R1" gate="G$1" pin="1"/>
+<wire x1="114.3" y1="38.1" x2="114.3" y2="35.56" width="0.1524" layer="91"/>
+<pinref part="GND13" gate="1" pin="GND"/>
+</segment>
 </net>
 <net name="+3V3" class="0">
@@
 <pinref part="R3" gate="G$1" pin="2"/>
 <pinref part="+3V4" gate="G$1" pin="+3V3"/>
-<wire x1="30.48" y1="76.2" x2="30.48" y2="78.74" width="0.1524" layer="91"/>
-<wire x1="30.48" y1="78.74" x2="38.1" y2="78.74" width="0.1524" layer="91"/>
-<pinref part="R1" gate="G$1" pin="2"/>
-<wire x1="38.1" y1="78.74" x2="45.72" y2="78.74" width="0.1524" layer="91"/>
-<wire x1="45.72" y1="78.74" x2="45.72" y2="76.2" width="0.1524" layer="91"/>
-<junction x="45.72" y="78.74"/>
+<wire x1="30.48" y1="71.12" x2="30.48" y2="73.66" width="0.1524" layer="91"/>
+<wire x1="30.48" y1="73.66" x2="38.1" y2="73.66" width="0.1524" layer="91"/>
+<wire x1="38.1" y1="73.66" x2="38.1" y2="76.2" width="0.1524" layer="91"/>
 <pinref part="R2" gate="G$1" pin="2"/>
-<wire x1="38.1" y1="78.74" x2="38.1" y2="76.2" width="0.1524" layer="91"/>
-<junction x="38.1" y="78.74"/>
+<wire x1="38.1" y1="73.66" x2="38.1" y2="71.12" width="0.1524" layer="91"/>
+<junction x="38.1" y="73.66"/>
+</segment>
+<segment>
+<pinref part="MCP2515" gate="D" pin="RESET"/>
+<wire x1="50.8" y1="63.5" x2="45.72" y2="63.5" width="0.1524" layer="91"/>
+<wire x1="45.72" y1="63.5" x2="45.72" y2="66.04" width="0.1524" layer="91"/>
+<pinref part="+3V5" gate="G$1" pin="+3V3"/>
 </segment>
 </net>
@@
 <pinref part="R2" gate="G$1" pin="1"/>
 <wire x1="50.8" y1="58.42" x2="38.1" y2="58.42" width="0.1524" layer="91"/>
-<wire x1="38.1" y1="58.42" x2="38.1" y2="66.04" width="0.1524" layer="91"/>
+<wire x1="38.1" y1="58.42" x2="38.1" y2="60.96" width="0.1524" layer="91"/>
 <label x="40.64" y="58.42" size="1.778" layer="95"/>
 </segment>
@@
 </segment>
 </net>
-<net name="N$1" class="0">
-<segment>
-<pinref part="MCP2515" gate="D" pin="RESET"/>
-<pinref part="R1" gate="G$1" pin="1"/>
-<wire x1="50.8" y1="63.5" x2="45.72" y2="63.5" width="0.1524" layer="91"/>
-<wire x1="45.72" y1="63.5" x2="45.72" y2="66.04" width="0.1524" layer="91"/>
-</segment>
-</net>
 <net name="CS" class="0">
 <segment>
@@
 <pinref part="R3" gate="G$1" pin="1"/>
 <wire x1="50.8" y1="53.34" x2="30.48" y2="53.34" width="0.1524" layer="91"/>
-<wire x1="30.48" y1="53.34" x2="30.48" y2="66.04" width="0.1524" layer="91"/>
+<wire x1="30.48" y1="53.34" x2="30.48" y2="60.96" width="0.1524" layer="91"/>
 <label x="40.64" y="53.34" size="1.778" layer="95"/>
 </segment>
@@
 </segment>
 </net>
-<net name="N$5" class="0">
+<net name="TXCAN" class="0">
 <segment>
 <pinref part="MCP2515" gate="D" pin="TXCAN"/>
@@
 </segment>
 </net>
-<net name="N$6" class="0">
+<net name="RXCAN" class="0">
 <segment>
 <pinref part="MCP2515" gate="D" pin="RXCAN"/>
-<pinref part="R4" gate="G$1" pin="2"/>
 <wire x1="83.82" y1="55.88" x2="101.6" y2="55.88" width="0.1524" layer="91"/>
 <pinref part="R5" gate="G$1" pin="1"/>
@@
 <wire x1="101.6" y1="55.88" x2="101.6" y2="53.34" width="0.1524" layer="91"/>
 <junction x="101.6" y="55.88"/>
-</segment>
-</net>
-<net name="N$7" class="0">
-<segment>
 <pinref part="R4" gate="G$1" pin="1"/>
+</segment>
+</net>
+<net name="RXCAN_5V" class="0">
+<segment>
 <pinref part="MCP2551" gate="G$1" pin="RXD"/>
 <wire x1="114.3" y1="55.88" x2="116.84" y2="55.88" width="0.1524" layer="91"/>
+<pinref part="R4" gate="G$1" pin="2"/>
 </segment>
 </net>
@@
 </segment>
 </net>
+<net name="N$1" class="0">
+<segment>
+<pinref part="MCP2551" gate="G$1" pin="RS"/>
+<pinref part="R1" gate="G$1" pin="2"/>
+<wire x1="116.84" y1="48.26" x2="114.3" y2="48.26" width="0.1524" layer="91"/>
+</segment>
+</net>
